File: Prova2.kicad_sch (KiCad schematic)
At the start: 1 part

Commit message: Nuove modifiche
Parts:
- added J?: Conn_01x08, symbol Connector_Generic:Conn_01x08
- added U?: BUF602xDBV, Package_TO_SOT_SMD:SOT-23-5, symbol Amplifier_Buffer:BUF602xDBV
- added U?: LM6321H, Package_TO_SOT_THT:TO-5-8, symbol Amplifier_Buffer:LM6321H
Changed lines of the file:
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@@
     (pin "9")
+  )
+  (symbol (lib_id "Amplifier_Buffer:BUF602xDBV") (at 104.14 82.55 0) (unit 1)
+    (in_bom yes) (on_board yes) (fields_autoplaced)
+    (property "Reference" "U?" (id 0) (at 116.84 77.851 0))
+    (property "Value" "BUF602xDBV" (id 1) (at 116.84 80.391 0))
+    (property "Footprint" "Package_TO_SOT_SMD:SOT-23-5" (id 2) (at 104.14 90.17 0)
+      (effects (font (size 1.27 1.27)) hide)
+    )
+    (property "Datasheet" "http://www.ti.com/lit/ds/symlink/buf602.pdf" (id 3) (at 104.14 82.55 0)
+      (effects (font (size 1.27 1.27)) hide)
+    )
+    (pin "1")
+    (pin "2")
+    (pin "3")
+    (pin "4")
+    (pin "5")
+  )
+  (symbol (lib_id "Connector_Generic:Conn_01x08") (at 212.09 83.82 0) (unit 1)
+    (in_bom yes) (on_board yes) (fields_autoplaced)
+    (property "Reference" "J?" (id 0) (at 214.63 83.8199 0)
+      (effects (font (size 1.27 1.27)) (justify left))
+    )
+    (property "Value" "Conn_01x08" (id 1) (at 214.63 86.3599 0)
+      (effects (font (size 1.27 1.27)) (justify left))
+    )
+    (property "Footprint" "" (id 2) (at 212.09 83.82 0)
+      (effects (font (size 1.27 1.27)) hide)
+    )
+    (property "Datasheet" "~" (id 3) (at 212.09 83.82 0)
+      (effects (font (size 1.27 1.27)) hide)
+    )
+    (pin "1")
+    (pin "2")
+    (pin "3")
+    (pin "4")
+    (pin "5")
+    (pin "6")
+    (pin "7")
+    (pin "8")
+  )
+  (symbol (lib_id "Amplifier_Buffer:LM6321H") (at 104.14 111.76 0) (unit 1)
+    (in_bom yes) (on_board yes) (fields_autoplaced)
+    (property "Reference" "U?" (id 0) (at 115.57 107.061 0))
+    (property "Value" "LM6321H" (id 1) (at 115.57 109.601 0))
+    (property "Footprint" "Package_TO_SOT_THT:TO-5-8" (id 2) (at 104.14 111.76 0)
+      (effects (font (size 1.27 1.27)) hide)
+    )
+    (property "Datasheet" "http://www.electronica60norte.com/mwfls/pdf/LM6221.pdf" (id 3) (at 104.14 111.76 0)
+      (effects (font (size 1.27 1.27)) hide)
+    )
+    (pin "1")
+    (pin "2")
+    (pin "3")
+    (pin "4")
+    (pin "5")
+    (pin "6")
+    (pin "7")
+    (pin "8")
   )
   (sheet_instances
@@
   )
   (symbol_instances
+    (path "/a53bb674-d6aa-4eed-b93d-2ee96e16b6d0"
+      (reference "J?") (unit 1) (value "Conn_01x08") (footprint "")
+    )
     (path "/0636e779-7442-4c24-a48f-6ad603dfc306"
       (reference "U?") (unit 1) (value "74AHC240") (footprint "")
     )
+    (path "/1b519627-3e8c-46d4-aac4-bcb4a32c08ff"
+      (reference "U?") (unit 1) (value "BUF602xDBV") (footprint "Package_TO_SOT_SMD:SOT-23-5")
+    )
+    (path "/abe47316-6765-4e23-b538-2ddd137d4326"
+      (reference "U?") (unit 1) (value "LM6321H") (footprint "Package_TO_SOT_THT:TO-5-8")
+    )
   )

Commit message: name
Parts:
- added U?: 74AHC273, symbol 74xx:74AHC273
Changed lines of the file:
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@@
     (pin "5")
+  )
+  (symbol (lib_id "74xx:74AHC273") (at 238.76 54.61 0) (unit 1)
+    (in_bom yes) (on_board yes) (fields_autoplaced)
+    (property "Reference" "U?" (id 0) (at 240.7794 34.29 0)
+      (effects (font (size 1.27 1.27)) (justify left))
+    )
+    (property "Value" "74AHC273" (id 1) (at 240.7794 36.83 0)
+      (effects (font (size 1.27 1.27)) (justify left))
+    )
+    (property "Footprint" "" (id 2) (at 238.76 54.61 0)
+      (effects (font (size 1.27 1.27)) hide)
+    )
+    (property "Datasheet" "https://assets.nexperia.com/documents/data-sheet/74AHC_AHCT273.pdf" (id 3) (at 238.76 54.61 0)
+      (effects (font (size 1.27 1.27)) hide)
+    )
+    (pin "1")
+    (pin "10")
+    (pin "11")
+    (pin "12")
+    (pin "13")
+    (pin "14")
+    (pin "15")
+    (pin "16")
+    (pin "17")
+    (pin "18")
+    (pin "19")
+    (pin "2")
+    (pin "20")
+    (pin "3")
+    (pin "4")
+    (pin "5")
+    (pin "6")
+    (pin "7")
+    (pin "8")
+    (pin "9")
   )
   (symbol (lib_id "Connector_Generic:Conn_01x08") (at 212.09 83.82 0) (unit 1)
@@
       (reference "U?") (unit 1) (value "BUF602xDBV") (footprint "Package_TO_SOT_SMD:SOT-23-5")
     )
+    (path "/288f44a3-9202-48ff-b843-7ecb952e643d"
+      (reference "U?") (unit 1) (value "74AHC273") (footprint "")
+    )
     (path "/abe47316-6765-4e23-b538-2ddd137d4326"
